Commit message: Rotate arm base 180° to match physical mounting
실제 로봇팔 베이스가 180° 회전 장착됨 → arm_base_joint rpy 0→π 반영
joint1=-3.141(unified.py HOME)로 보정하면 팔이 엘리베이터 방향을 향함

Co-Authored-By: Claude Sonnet 4.6 <noreply@anthropic.com>

File: urdf/mobile_manipulator.urdf.xacro (robot description, xacro)
@@ -98,5 +98,5 @@
     <child link="$(arg prefix)link1"/>
     <!-- 차체 상단(0.069) + 프로파일(0.65) + 상판(0.005) = 0.724 -->
-    <origin xyz="-0.12757 0.0 0.724" rpy="0 0 0"/>
+    <origin xyz="-0.12757 0.0 0.724" rpy="0 0 3.14159"/>
   </joint>
 </robot>
